File: Sensing.kicad_sch (KiCad schematic)
At the start: 20 parts, among them Q1 ZXMP2120FFTA, Q2 ZXMP2120FFTA, U1 LTC4368CMS-1#PBF, U2 INA226AIDGSR, U3 MCP9808T-E/MS, U7 MCP9808T-E/MS, U8 MCP9808T-E/MS

Commit message: Added actuation circuitry
Connections:
- net TEMP1_ALERT: now reaches U3.3 (ALERT)
- net TEMP3_ALERT: now reaches U7.3 (ALERT)
- net TEMP2_ALERT: now reaches U8.3 (ALERT)
Changed lines of the file:
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@@
 	(generator "eeschema")
 	(generator_version "10.0")
-	(paper "A4")
+	(paper "A3")
 	(rectangle
 		(start 13.97 16.51)
@@
 	(wire
 		(pts
+			(xy 186.69 35.56) (xy 196.85 35.56)
+		)
+		(stroke
+			(width 0)
+			(type default)
+		)
+	)
+	(wire
+		(pts
 			(xy 97.79 43.18) (xy 97.79 76.2)
 		)
@@
 	(wire
 		(pts
+			(xy 187.96 85.09) (xy 198.12 85.09)
+		)
+		(stroke
+			(width 0)
+			(type default)
+		)
+	)
+	(wire
+		(pts
 			(xy 85.09 48.26) (xy 85.09 49.53)
 		)
@@
 		(pts
 			(xy 96.52 107.95) (xy 96.52 105.41)
+		)
+		(stroke
+			(width 0)
+			(type default)
+		)
+	)
+	(wire
+		(pts
+			(xy 186.69 60.96) (xy 196.85 60.96)
 		)
 		(stroke
@@
 		)
 	)
+	(label "TEMP3_ALERT"
+		(at 187.96 85.09 0)
+		(effects
+			(font
+				(size 1.27 1.27)
+			)
+			(justify left bottom)
+		)
+	)
 	(label "VSENSE_ALERT"
 		(at 85.09 132.08 0)
@@
 		)
 	)
+	(label "TEMP2_ALERT"
+		(at 186.69 60.96 0)
+		(effects
+			(font
+				(size 1.27 1.27)
+			)
+			(justify left bottom)
+		)
+	)
 	(label "VSENSE_SDA"
 		(at 85.09 127 0)
@@
 		(effects
 			(font
+				(size 1.27 1.27)
+			)
+			(justify left bottom)
+		)
+	)
+	(label "TEMP1_ALERT"
+		(at 186.69 35.56 0)
+		(effects
+			(font
